Commit message: adding file

File: src/my_robot/urdf/my_robot.xacro (robot description, xacro)
@@ -55,3 +55,26 @@
                                                     </visual>
                                                   </link>
+   <link name="right_wheel">
+    <visual>
+      <origin xyz="0.0 0.0 0.0" rpy="0.0 0.0 0.0"/>
+      <geometry>
+        <cylinder length="0.05" radius="0.1"/>
+      </geometry>
+    </visual>
+    <collision>
+      <origin xyz="0.0 0.0 0.0" rpy="0.0 0.0 0.0"/>
+      <geometry>
+        <cylinder length="0.05" radius="0.1"/>
+      </geometry>
+    </collision>
+    <inertial>
+      <origin xyz="0.0 0.0 0.0" rpy="0.0 1.5707 1.5707"/>
+      <mass value="5"/>
+      <inertia
+          ixx="0.1" ixy="0" ixz="0"
+          iyy="0.1" iyz="0"
+          izz="0.1"
+      />
+    </inertial>
+  </link>
 </robot>

Commit message: updates

File: src/my_robot/urdf/my_robot.xacro (robot description, xacro)
@@ -55,7 +55,46 @@
                                                     </visual>
                                                   </link>
+  <joint type="continuous" name="right_wheel_hinge">
+    <origin xyz="0 0.13 0" rpy="0 0 0"/>
+    <child link="right_wheel"/>
+    <parent link="chassis"/>
+    <axis xyz="0 0.12 0" rpy="0 0 0"/>
+    <limit effort="10000" velocity="1000"/>
+    <dynamics damping="1.0" friction="1.0"/>
+  </joint>
    <link name="right_wheel">
     <visual>
+      <origin xyz="0.0 0.0 0.0" rpy="1.5707 0.0 0"/>
+      <geometry>
+        <cylinder length="0.05" radius="0.1"/>
+      </geometry>
+    </visual>
+    <collision>
       <origin xyz="0.0 0.0 0.0" rpy="0.0 0.0 0.0"/>
+      <geometry>
+        <cylinder length="0.05" radius="0.1"/>
+      </geometry>
+    </collision>
+    <inertial>
+      <origin xyz="0.0 0.0 0.0" rpy="0.0 1.5707 1.5707"/>
+      <mass value="5"/>
+      <inertia
+          ixx="0.1" ixy="0" ixz="0"
+          iyy="0.1" iyz="0"
+          izz="0.1"
+      />
+    </inertial>
+  </link>
+  <joint type="continuous" name="left_wheel_hinge">
+    <origin xyz="0 -0.13 0" rpy="0 0 0"/>
+    <child link="left_wheel"/>
+    <parent link="chassis"/>
+    <axis xyz="0 0.12 0" rpy="0 0 0"/>
+    <limit effort="10000" velocity="1000"/>
+    <dynamics damping="1.0" friction="1.0"/>
+  </joint>
+   <link name="left_wheel">
+    <visual>
+      <origin xyz="0.0 0.0 0.0" rpy="1.5707 0.0 0"/>
       <geometry>
         <cylinder length="0.05" radius="0.1"/>

Commit message: updates

File: src/my_robot/urdf/my_robot.xacro (robot description, xacro)
@@ -77,5 +77,5 @@
     </collision>
     <inertial>
-      <origin xyz="0.0 0.0 0.0" rpy="0.0 1.5707 1.5707"/>
+      <origin xyz="0.0 0.0 0.0" rpy="0.0 0 0"/>
       <mass value="5"/>
       <inertia
@@ -84,4 +84,44 @@
           izz="0.1"
       />
+    </inertial>
+  </link>
+  <joint type="fixed" name="camera_joint">
+    <origin xyz="0.2 0 0" rpy="0 0 0"/>
+    <child link="camera"/>
+    <parent link="chassis"/>
+    <axis xyz="0 0.1 0" rpy="0 0 0"/>
+    <limit effort="10000" velocity="1000"/>
+    <dynamics damping="1.0" friction="1.0"/>
+  </joint>
+   <link name="camera">
+    <visual>
+      <origin xyz="0.0 0.0 0.0" rpy="0 0 0"/>
+      <geometry>
+        <box>
+        <size>0.05 0.05 0.05</size>
+        </box>
+      </geometry>
+    </visual>
+    <collision>
+      <origin xyz="0.0 0.0 0.0" rpy="0.0 0.0 0.0"/>
+      <geometry>
+        <box>
+        <size>0.05 0.05 0.05</size>
+        </box>
+      </geometry>
+    </collision>
+    <inertial>
+      <origin xyz="0.0 0.0 0.0" rpy="0.0 0 0"/>
+      <mass value="0.1"/>
+      <inertia
+          ixx="0.000001" ixy="0" ixz="0"
+          iyy="0.000001" iyz="0"
+          izz="0.000001"
+      />
+      <geometry>
+        <box>
+        <size>0.05 0.05 0.05</size>
+        </box>
+      </geometry>
     </inertial>
   </link>

Commit message: gazebo plugin files

File: src/my_robot/urdf/my_robot.xacro (robot description, xacro)
@@ -90,5 +90,5 @@
     <child link="camera"/>
     <parent link="chassis"/>
-    <axis xyz="0 0.1 0" rpy="0 0 0"/>
+    <axis xyz="0 1 0" rpy="0 0 0"/>
     <limit effort="10000" velocity="1000"/>
     <dynamics damping="1.0" friction="1.0"/>
@@ -97,17 +97,13 @@
     <visual>
       <origin xyz="0.0 0.0 0.0" rpy="0 0 0"/>
-      <geometry>
-        <box>
-        <size>0.05 0.05 0.05</size>
-        </box>
-      </geometry>
+        <geometry>
+          <box size=".05 .05 .05"/>
+        </geometry>
     </visual>
     <collision>
       <origin xyz="0.0 0.0 0.0" rpy="0.0 0.0 0.0"/>
-      <geometry>
-        <box>
-        <size>0.05 0.05 0.05</size>
-        </box>
-      </geometry>
+        <geometry>
+          <box size=".05 .05 .05"/>
+        </geometry>
     </collision>
     <inertial>
@@ -119,9 +115,7 @@
           izz="0.000001"
       />
-      <geometry>
-        <box>
-        <size>0.05 0.05 0.05</size>
-        </box>
-      </geometry>
+        <geometry>
+          <box size=".05 .05 .05"/>
+        </geometry>
     </inertial>
   </link>
@@ -157,3 +151,37 @@
     </inertial>
   </link>
+  <joint type="fixed" name="hokuyo_joint">
+    <origin xyz="0.15 0 0.1" rpy="0 0 0"/>
+    <child link="hokuyo"/>
+    <parent link="chassis"/>
+    <axis xyz="0 1 0" rpy="0 0 0"/>
+    <limit effort="10000" velocity="1000"/>
+    <dynamics damping="1.0" friction="1.0"/>
+  </joint>
+   <link name="hokuyo">
+    <visual>
+      <origin xyz="0.0 0.0 0.0" rpy="0 0 0"/>
+        <geometry>
+          <box size=".05 .05 .05"/>
+        </geometry>
+    </visual>
+    <collision>
+      <origin xyz="0.0 0.0 0.0" rpy="0.0 0.0 0.0"/>
+        <geometry>
+          <box size=".05 .05 .05"/>
+        </geometry>
+    </collision>
+    <inertial>
+      <origin xyz="0.0 0.0 0.0" rpy="0.0 0 0"/>
+      <mass value="0.1"/>
+      <inertia
+          ixx="0.000001" ixy="0" ixz="0"
+          iyy="0.000001" iyz="0"
+          izz="0.000001"
+      />
+        <geometry>
+          <box size=".05 .05 .05"/>
+        </geometry>
+    </inertial>
+  </link>
 </robot>
